File: collectorunit/hw/power.sch (KiCad schematic (older format))
At the start: 15 parts, among them CON1 BARREL_JACK, P1 CONN_01X02, U1 LT3652

Commit message: Further work on the power unit
Parts:
- added C4: 10uF, symbol C
- added P2: LOAD, symbol CONN_01X02
- D4: value D_Schottky_Small -> Schottky_Flyback
- P1: value CONN_01X02 -> BATTREY
- R2: value 666K -> 66K
Connections:
- net +6V: now also C4.1
- net CHRG: now also C3.1, D3.2 (A), R4.1, R6.1, U1.9 (BAT), P2.1 (P1); no longer L1.2, R6.2, U1.10 (SENSE)
- net GND: now also C4.2, P2.2 (P2); no longer P1.2 (P2)
- net at U1.4 (~CHRG): now also D2.1 (K); no longer D1.1 (K)
- net at U1.5 (~FAULT): now also D1.1 (K); no longer D2.1 (K)
- new net: L1.2, R6.2, U1.10 (SENSE)
Other:
- note added: "This node becomes \nGND when SW is OFF"
- moved on the sheet: D1, D2, P1, R2, R3
Changed lines of the file:
@@
 L R R2
 U 1 1 56BF647F
-P 4150 2900
-F 0 "R2" V 4230 2900 50  0000 C CNN
-F 1 "666K" V 4150 2900 50  0000 C CNN
-F 2 "" V 4080 2900 50  0000 C CNN
-F 3 "" H 4150 2900 50  0000 C CNN
-	1    4150 2900
+P 4150 2950
+F 0 "R2" V 4230 2950 50  0000 C CNN
+F 1 "66K" V 4150 2950 50  0000 C CNN
+F 2 "" V 4080 2950 50  0000 C CNN
+F 3 "" H 4150 2950 50  0000 C CNN
+	1    4150 2950
 	1    0    0    -1
 $EndComp
@@
 L R R3
 U 1 1 56BF652A
-P 4150 3300
-F 0 "R3" V 4230 3300 50  0000 C CNN
-F 1 "100K" V 4150 3300 50  0000 C CNN
-F 2 "" V 4080 3300 50  0000 C CNN
-F 3 "" H 4150 3300 50  0000 C CNN
-	1    4150 3300
-	1    0    0    -1
-$EndComp
-$Comp
-L GND #PWR06
+P 4150 3250
+F 0 "R3" V 4230 3250 50  0000 C CNN
+F 1 "100K" V 4150 3250 50  0000 C CNN
+F 2 "" V 4080 3250 50  0000 C CNN
+F 3 "" H 4150 3250 50  0000 C CNN
+	1    4150 3250
+	1    0    0    -1
+$EndComp
+$Comp
+L GND #PWR7
 U 1 1 56BF68B8
 P 5000 4150
-F 0 "#PWR06" H 5000 3900 50  0001 C CNN
+F 0 "#PWR7" H 5000 3900 50  0001 C CNN
 F 1 "GND" H 5000 4000 50  0000 C CNN
 F 2 "" H 5000 4150 50  0000 C CNN
@@
 Text Notes 6000 3850 1    39   ~ 0
 4.2V FLT
-Text Notes 4050 3350 1    60   ~ 0
+Text Notes 4050 3250 1    39   ~ 0
 4.5V PEAK
 $Comp
 L CONN_01X02 P1
 U 1 1 56BF6DFB
-P 7550 3450
-F 0 "P1" H 7550 3600 50  0000 C CNN
-F 1 "CONN_01X02" V 7650 3450 50  0000 C CNN
-F 2 "" H 7550 3450 50  0000 C CNN
-F 3 "" H 7550 3450 50  0000 C CNN
-	1    7550 3450
+P 7550 3750
+F 0 "P1" H 7550 3900 50  0000 C CNN
+F 1 "BATTREY" V 7650 3750 50  0000 C CNN
+F 2 "" H 7550 3750 50  0000 C CNN
+F 3 "" H 7550 3750 50  0000 C CNN
+	1    7550 3750
 	1    0    0    -1
 $EndComp
@@
 $EndComp
 Wire Wire Line
-	4150 3050 4150 3150
-Wire Wire Line
-	4550 3100 4150 3100
+	4150 3100 4550 3100
 Connection ~ 4150 3100
 Wire Wire Line
-	2900 2500 4300 2500
-Wire Wire Line
-	4150 2750 4150 2500
+	2900 2500 3000 2500
+Wire Wire Line
+	3000 2500 3300 2500
+Wire Wire Line
+	3300 2500 4150 2500
+Wire Wire Line
+	4150 2500 4300 2500
+Wire Wire Line
+	4150 2800 4150 2500
 Connection ~ 4150 2500
 Wire Wire Line
 	4550 2950 4300 2950
 Wire Wire Line
-	4300 2500 4300 3250
-Wire Wire Line
-	5000 3950 5000 4150
-Wire Wire Line
-	4300 3250 4550 3250
-Connection ~ 4300 2950
+	5000 3950 5000 4000
+Wire Wire Line
+	5000 4000 5000 4100
+Wire Wire Line
+	5000 4100 5000 4150
 Wire Wire Line
 	4550 3750 4550 4000
 Wire Wire Line
-	4150 4000 5000 4000
+	4150 4000 4550 4000
+Wire Wire Line
+	4550 4000 5000 4000
 Connection ~ 5000 4000
 Wire Wire Line
@@
 Connection ~ 5800 3750
 Connection ~ 5000 4100
-Wire Wire Line
-	4150 3450 4150 4000
 Connection ~ 4550 4000
 Wire Wire Line
@@
 Connection ~ 5800 3450
 Wire Wire Line
-	5450 3450 6550 3450
+	5450 3450 5600 3450
+Wire Wire Line
+	5600 3450 5800 3450
+Wire Wire Line
+	5800 3450 6550 3450
+Wire Wire Line
+	6550 3450 6900 3450
+Wire Wire Line
+	6900 3450 7100 3450
+Wire Wire Line
+	7100 3450 7350 3450
+Wire Wire Line
+	7350 3450 7850 3450
 Wire Wire Line
 	6550 3150 5800 3150
@@
 	5800 3150 5800 3250
 Wire Wire Line
-	5800 4050 5800 4100
-Wire Wire Line
-	2900 4100 7350 4100
+	5800 4100 5800 4050
+Wire Wire Line
+	2900 4100 3300 4100
+Wire Wire Line
+	3300 4100 5000 4100
+Wire Wire Line
+	5000 4100 5800 4100
+Wire Wire Line
+	5800 4100 6550 4100
+Wire Wire Line
+	6550 4100 7850 4100
 Wire Wire Line
 	6550 3450 6550 3550
 Connection ~ 5800 4100
 Wire Wire Line
-	7350 4100 7350 3500
+	7350 3800 7350 4100
 Wire Wire Line
 	5450 3100 5600 3100
 Wire Wire Line
-	7350 2800 7350 3400
+	7350 3450 7350 3700
 $Comp
 L INDUCTOR_SMALL L1
@@
 $EndComp
 Wire Wire Line
-	5600 3050 5600 3200
+	5600 3050 5600 3100
+Wire Wire Line
+	5600 3100 5600 3200
 Wire Wire Line
 	5600 3400 5600 3450
@@
 	5450 2950 5450 2800
 Wire Wire Line
-	5450 2800 5850 2800
-Wire Wire Line
-	5600 2500 5600 2850
+	5450 2800 5600 2800
+Wire Wire Line
+	5600 2800 5850 2800
+Wire Wire Line
+	5600 2500 5600 2800
+Wire Wire Line
+	5600 2800 5600 2850
 Connection ~ 5600 2800
-Wire Wire Line
-	6350 2800 7350 2800
-Connection ~ 6550 2800
 $Comp
 L D_Schottky_Small D4
@@
 P 5950 2500
 F 0 "D4" H 5900 2580 50  0000 L CNN
-F 1 "D_Schottky_Small" H 5670 2420 50  0000 L CNN
+F 1 "Schottky_Flyback" H 5670 2420 50  0000 L CNN
 F 2 "" V 5950 2500 50  0000 C CNN
 F 3 "" V 5950 2500 50  0000 C CNN
@@
 	5850 2500 5600 2500
 $Comp
-L GND #PWR07
+L GND #PWR8
 U 1 1 56BF83E0
 P 6450 2550
-F 0 "#PWR07" H 6450 2300 50  0001 C CNN
+F 0 "#PWR8" H 6450 2300 50  0001 C CNN
 F 1 "GND" H 6450 2400 50  0000 C CNN
 F 2 "" H 6450 2550 50  0000 C CNN
@@
 L Led_Small D1
 U 1 1 56BF84FA
-P 3900 3550
-F 0 "D1" H 3850 3675 50  0000 L CNN
-F 1 "Led_Small" H 3725 3450 50  0000 L CNN
-F 2 "" V 3900 3550 50  0000 C CNN
-F 3 "" V 3900 3550 50  0000 C CNN
-	1    3900 3550
-	-1   0    0    1
+P 4400 4350
+F 0 "D1" H 4350 4500 50  0000 L CNN
+F 1 "Led_Small" H 4250 4600 50  0000 L CNN
+F 2 "" V 4400 4350 50  0000 C CNN
+F 3 "" V 4400 4350 50  0000 C CNN
+	1    4400 4350
+	0    1    1    0
 $EndComp
 $Comp
 L Led_Small D2
 U 1 1 56BF85B9
-P 3900 3800
-F 0 "D2" H 3850 3925 50  0000 L CNN
-F 1 "Led_Small" H 3725 3700 50  0000 L CNN
-F 2 "" V 3900 3800 50  0000 C CNN
-F 3 "" V 3900 3800 50  0000 C CNN
-	1    3900 3800
-	-1   0    0    1
-$EndComp
-Wire Wire Line
-	4000 3550 4300 3550
-Wire Wire Line
-	4300 3550 4300 3450
-Wire Wire Line
-	4300 3450 4550 3450
-Wire Wire Line
-	4550 3600 4300 3600
-Wire Wire Line
-	4300 3600 4300 3800
-Wire Wire Line
-	4300 3800 4000 3800
+P 4300 4350
+F 0 "D2" H 4250 4150 50  0000 L CNN
+F 1 "Led_Small" H 4150 4250 50  0000 L CNN
+F 2 "" V 4300 4350 50  0000 C CNN
+F 3 "" V 4300 4350 50  0000 C CNN
+	1    4300 4350
+	0    1    1    0
+$EndComp
 NoConn ~ 5450 3600
 Text Notes 8250 4400 2    39   ~ 0
 D3: average current greater than 0.1A, and reverse voltage greater than VIN(MAX)
-Text GLabel 3550 3800 0    39   Input ~ 0
+Text GLabel 4400 4650 3    39   Input ~ 0
 FAULT
-Text GLabel 3550 3550 0    39   Input ~ 0
+Text GLabel 4300 4650 3    39   Input ~ 0
 CHRG
-Wire Wire Line
-	3550 3550 3800 3550
-Wire Wire Line
-	3550 3800 3800 3800
-Text GLabel 7150 3300 0    39   Input ~ 0
+Text GLabel 6900 3250 1    39   Input ~ 0
 CHRG
-Text GLabel 7150 3150 0    39   Input ~ 0
+Text GLabel 7100 3250 1    39   Input ~ 0
 FAULT
-Wire Wire Line
-	7150 3150 7350 3150
-Connection ~ 7350 3150
-Wire Wire Line
-	7150 3300 7350 3300
-Connection ~ 7350 3300
 Wire Wire Line
 	2900 4100 2900 2700
 NoConn ~ 2900 2600
 $Comp
-L +6V #PWR08
+L +6V #PWR6
 U 1 1 56C06113
 P 3000 2350
-F 0 "#PWR08" H 3000 2200 50  0001 C CNN
+F 0 "#PWR6" H 3000 2200 50  0001 C CNN
 F 1 "+6V" H 3000 2490 50  0000 C CNN
 F 2 "" H 3000 2350 50  0000 C CNN
@@
 	3000 2350 3000 2500
 Connection ~ 3000 2500
+Wire Wire Line
+	4150 3400 4150 4000
+Wire Wire Line
+	4300 2500 4300 2950
+Wire Wire Line
+	4300 2950 4300 3250
+Wire Wire Line
+	4400 4450 4400 4650
+Wire Wire Line
+	4300 4650 4300 4450
+Wire Wire Line
+	4400 4250 4400 3600
+Wire Wire Line
+	4400 3600 4550 3600
+Wire Wire Line
+	4300 4250 4300 3450
+Wire Wire Line
+	4300 3450 4550 3450
+$Comp
+L C C4
+U 1 1 56C0A532
+P 3300 2750
+F 0 "C4" H 3325 2850 50  0000 L CNN
+F 1 "10uF" H 3325 2650 50  0000 L CNN
+F 2 "" H 3338 2600 50  0000 C CNN
+F 3 "" H 3300 2750 50  0000 C CNN
+	1    3300 2750
+	1    0    0    -1
+$EndComp
+Wire Wire Line
+	3300 2600 3300 2500
+Connection ~ 3300 2500
+Wire Wire Line
+	3300 2900 3300 4100
+Connection ~ 3300 4100
+Wire Wire Line
+	6550 2800 6350 2800
+Connection ~ 6550 3450
+$Comp
+L CONN_01X02 P2
+U 1 1 56C0AE90
+P 8050 3750
+F 0 "P2" H 8050 3900 50  0000 C CNN
+F 1 "LOAD" V 8150 3750 50  0000 C CNN
+F 2 "" H 8050 3750 50  0000 C CNN
+F 3 "" H 8050 3750 50  0000 C CNN
+	1    8050 3750
+	1    0    0    -1
+$EndComp
+Wire Wire Line
+	7850 3450 7850 3700
+Connection ~ 7350 3450
+Wire Wire Line
+	7850 4100 7850 3800
+Wire Wire Line
+	6900 3250 6900 3450
+Connection ~ 6900 3450
+Wire Wire Line
+	7100 3250 7100 3450
+Connection ~ 7100 3450
+Wire Wire Line
+	4300 3250 4550 3250
+Connection ~ 4300 2950
+Text Notes 5700 2450 2    39   ~ 0
+This node becomes \nGND when SW is OFF
 $EndSCHEMATC
