File: collectorunit/hw/wscollectorunit.sch (KiCad schematic (older format))
At the start: 9 parts

Commit message: Working on the power unit
Parts:
- removed SR?: DS18B20, symbol DS18B20
- gave numbers to parts that had none: 8
Changed lines of the file:
@@
 LIBS:contrib
 LIBS:valves
-LIBS:AmbientTempNode-cache
+LIBS:w_analog
+LIBS:wscollectorunit-cache
 EELAYER 25 0
 EELAYER END
 $Descr A4 11693 8268
 encoding utf-8
-Sheet 1 1
+Sheet 1 2
 Title ""
 Date ""
@@
 $EndDescr
 $Comp
-L ATMEGA8-P IC?
+L ATMEGA8-P IC1
 U 1 1 569A3BA5
 P 3450 3250
-F 0 "IC?" H 2700 4550 50  0000 L BNN
+F 0 "IC1" H 2700 4550 50  0000 L BNN
 F 1 "ATMEGA8-P" H 3950 1800 50  0000 L BNN
 F 2 "DIL28" H 3450 3250 50  0000 C CIN
@@
 $EndComp
 $Comp
-L ADAFRUIT-LCD16x2-RGB DS?
+L ADAFRUIT-LCD16x2-RGB DS1
 U 1 1 569A4811
 P 6750 3700
-F 0 "DS?" H 5850 4100 50  0000 C CNN
+F 0 "DS1" H 5850 4100 50  0000 C CNN
 F 1 "ADAFRUIT-LCD16x2-RGB" H 7250 4100 50  0000 C CNN
 F 2 "HD44780" H 6750 3650 50  0000 C CIN
@@
 $EndComp
 $Comp
-L SW_PUSH SW?
+L SW_PUSH SW2
 U 1 1 56ABA85F
 P 4950 4950
-F 0 "SW?" H 5100 5060 50  0000 C CNN
+F 0 "SW2" H 5100 5060 50  0000 C CNN
 F 1 "SW_PUSH" H 4950 4870 50  0000 C CNN
 F 2 "" H 4950 4950 50  0000 C CNN
@@
 $EndComp
 $Comp
-L GND #PWR?
+L GND #PWR01
 U 1 1 56ABAB0F
 P 4950 5250
-F 0 "#PWR?" H 4950 5000 50  0001 C CNN
+F 0 "#PWR01" H 4950 5000 50  0001 C CNN
 F 1 "GND" H 4950 5100 50  0000 C CNN
 F 2 "" H 4950 5250 50  0000 C CNN
@@
 $EndComp
 $Comp
-L BS170 Q?
+L BS170 Q1
 U 1 1 56AFEABB
 P 5700 2100
-F 0 "Q?" H 5900 2175 50  0000 L CNN
+F 0 "Q1" H 5900 2175 50  0000 L CNN
 F 1 "BS170" H 5900 2100 50  0000 L CNN
 F 2 "TO-92" H 5900 2025 50  0000 L CIN
@@
 	4450 2150 5500 2150
 $Comp
-L +5V #PWR?
+L +5V #PWR02
 U 1 1 56AFED9B
 P 750 900
-F 0 "#PWR?" H 750 750 50  0001 C CNN
+F 0 "#PWR02" H 750 750 50  0001 C CNN
 F 1 "+5V" H 750 1040 50  0000 C CNN
 F 2 "" H 750 900 50  0000 C CNN
@@
 Connection ~ 1500 1100
 $Comp
-L R R?
+L R R1
 U 1 1 56AFEE34
 P 2350 1650
-F 0 "R?" V 2430 1650 50  0000 C CNN
+F 0 "R1" V 2430 1650 50  0000 C CNN
 F 1 "R" V 2350 1650 50  0000 C CNN
 F 2 "" V 2280 1650 50  0000 C CNN
@@
 Connection ~ 2350 1100
 $Comp
-L C C?
+L C C1
 U 1 1 56AFEF10
 P 2350 3400
-F 0 "C?" H 2375 3500 50  0000 L CNN
+F 0 "C1" H 2375 3500 50  0000 L CNN
 F 1 "C" H 2375 3300 50  0000 L CNN
 F 2 "" H 2388 3250 50  0000 C CNN
@@
 Connection ~ 2350 2150
 $Comp
-L GND #PWR?
+L GND #PWR03
 U 1 1 56AFF0E6
 P 2350 3700
-F 0 "#PWR?" H 2350 3450 50  0001 C CNN
+F 0 "#PWR03" H 2350 3450 50  0001 C CNN
 F 1 "GND" H 2350 3550 50  0000 C CNN
 F 2 "" H 2350 3700 50  0000 C CNN
@@
 	2350 3700 2350 3550
 $Comp
-L SW_PUSH SW?
+L SW_PUSH SW1
 U 1 1 56AFF14A
 P 1900 3250
-F 0 "SW?" H 2050 3360 50  0000 C CNN
+F 0 "SW1" H 2050 3360 50  0000 C CNN
 F 1 "SW_PUSH" H 1900 3170 50  0000 C CNN
 F 2 "" H 1900 3250 50  0000 C CNN
@@
 $EndComp
 $Comp
-L GND #PWR?
+L GND #PWR04
 U 1 1 56AFF20C
 P 1900 3700
-F 0 "#PWR?" H 1900 3450 50  0001 C CNN
+F 0 "#PWR04" H 1900 3450 50  0001 C CNN
 F 1 "GND" H 1900 3550 50  0000 C CNN
 F 2 "" H 1900 3700 50  0000 C CNN
@@
 	1900 3550 1900 3700
 $Comp
-L DS18B20 SR?
+L DS18B20 SR1
 U 1 1 56AFFE0E
 P 7950 2650
-F 0 "SR?" H 7950 2750 60  0000 C CNN
+F 0 "SR1" H 7950 2750 60  0000 C CNN
 F 1 "DS18B20" H 7950 2850 60  0000 C CNN
 F 2 "" H 7950 2650 60  0000 C CNN
@@
 $EndComp
 $Comp
-L DS18B20 SR?
-U 1 1 56AFFF27
-P 7950 2150
-F 0 "SR?" H 7950 2250 60  0000 C CNN
-F 1 "DS18B20" H 7950 2350 60  0000 C CNN
-F 2 "" H 7950 2150 60  0000 C CNN
-F 3 "" H 7950 2150 60  0000 C CNN
-	1    7950 2150
-	0    1    1    0
-$EndComp
-$Comp
-L GND #PWR?
+L GND #PWR05
 U 1 1 56AFFFA4
 P 7450 3250
-F 0 "#PWR?" H 7450 3000 50  0001 C CNN
+F 0 "#PWR05" H 7450 3000 50  0001 C CNN
 F 1 "GND" H 7450 3100 50  0000 C CNN
 F 2 "" H 7450 3250 50  0000 C CNN
@@
 $EndComp
 Wire Wire Line
-	7550 2050 7450 2050
-Wire Wire Line
-	7450 2050 7450 3250
+	4450 2650 7550 2650
 Wire Wire Line
 	7550 2750 7450 2750
+Wire Wire Line
+	7450 2550 7450 3250
+Wire Wire Line
+	7550 2550 7450 2550
 Connection ~ 7450 2750
-Wire Wire Line
-	7550 2550 7450 2550
-Connection ~ 7450 2550
-Wire Wire Line
-	7550 2250 7450 2250
-Connection ~ 7450 2250
-Wire Wire Line
-	4450 2650 7550 2650
-Wire Wire Line
-	7550 2150 7300 2150
-Wire Wire Line
-	7300 2150 7300 2650
-Connection ~ 7300 2650
+$Sheet
+S 9750 750  750  800
+U 56BF63B4
+F0 "Sheet56BF63B3" 60
+F1 "power.sch" 60
+$EndSheet
 $EndSCHEMATC
