File: lt3652_breakout/lt3652_breakout.sch (KiCad schematic (older format))
At the start: 4 parts, among them P1 CONN_01X06, P2 CONN_01X06, P3 GND, U1 LT3652

Commit message: WIP on LT3652 breakout
Parts:
- removed P1: CONN_01X06, Pin_Headers:Pin_Header_Straight_1x06, symbol CONN_01X06
- added C1: 0.68uF, Capacitors_ThroughHole:C_Disc_D3_P2.5, symbol C
- added C2: 10uF, Capacitors_ThroughHole:C_Disc_D3_P2.5, symbol C
- added C3: 10uF, Capacitors_ThroughHole:C_Disc_D3_P2.5, symbol C_Small
- added CON1: SLR PNL, Connect:JACK_ALIM, symbol BARREL_JACK
- added D1: 3mm GRN, LEDs:LED-3MM, symbol Led_Small
- added D2: 3mm RED, LEDs:LED-3MM, symbol Led_Small
- added JP1: SHDN OPT, Pin_Headers:Pin_Header_Straight_1x03, symbol JUMPER3
- added JP2: TIMER OPT, Pin_Headers:Pin_Header_Straight_1x03, symbol JUMPER3
- added JP3: VREG OPT, Pin_Headers:Pin_Header_Straight_1x03, symbol JUMPER3
- added P1: OUT LEFT, Pin_Headers:Pin_Header_Straight_1x03, symbol CONN_01X03
- added R1, R2: 220, Resistors_ThroughHole:Resistor_Horizontal_RM7mm, symbol R_Small
- P2: value CONN_01X06 -> OUT RIGHT
Connections:
- net labels added: GND, VREG
- net labels removed: BAT, BOOST, CHRG, FAULT, NTC, SENSE, SW, VFB, VIN_REG
- wire segments 25 -> 53
- no-connect marks 0 -> 1

Commit message: Started work on Rev 0.2, with the aim of using trimmer to configure the LT3652
Parts:
- added SW?: GRAYHILL_76SC04T, symbol GRAYHILL_76SC04T
Changed lines of the file:
@@
 Wire Wire Line
 	2800 2075 2925 2075
+$Comp
+L GRAYHILL_76SC04T SW?
+U 1 1 56C3C744
+P 6700 1525
+F 0 "SW?" H 6500 2275 50  0000 C CNN
+F 1 "GRAYHILL_76SC04T" H 6750 2375 50  0000 C CNN
+F 2 "" H 6700 2125 50  0000 C CNN
+F 3 "" H 6700 2125 50  0000 C CNN
+	1    6700 1525
+	-1   0    0    1
+$EndComp
 $EndSCHEMATC

Commit message: WIP on Rev 0.2
Parts:
- removed C1: 0.68uF, Capacitors_ThroughHole:C_Disc_D3_P2.5, symbol C
- removed JP1: SHDN OPT, Pin_Headers:Pin_Header_Straight_1x03, symbol JUMPER3
- removed JP3: VREG OPT, Pin_Headers:Pin_Header_Straight_1x03, symbol JUMPER3
- removed P1: OUT LEFT, Pin_Headers:Pin_Header_Straight_1x03, symbol CONN_01X03
- removed P2: OUT RIGHT, Pin_Headers:Pin_Header_Straight_1x06, symbol CONN_01X06
- removed P3: GND, Pin_Headers:Pin_Header_Straight_1x01, symbol CONN_01X01
- removed SW?: GRAYHILL_76SC04T, symbol GRAYHILL_76SC04T
- added C?: CTRIM, symbol CTRIM
- added C?: 1uF, Capacitors_SMD:C_0603_HandSoldering, symbol C_Small
- added D?: D_Small, symbol D_Small
- added P1: CONN_01X09, Pin_Headers:Pin_Header_Straight_1x09, symbol CONN_01X09
- added RV1, RV2, RV?: POT, bourns_trim_pots:Bourns_3362P_Trimmer, symbol POT
- added W1, W2: TEST_1P, pcb_test_points:KEYSTONE_5016_PCB_Test_Point, symbol TEST_1P
- C2, C3: footprint Capacitors_ThroughHole:C_Disc_D3_P2.5 -> Capacitors_SMD:C_0603_HandSoldering
- D1, D2: footprint LEDs:LED-3MM -> LEDs:LED_0603
- R1, R2: footprint Resistors_ThroughHole:Resistor_Horizontal_RM7mm -> Resistors_SMD:R_0603_HandSoldering
Connections:
- net labels added: VIN_REG
- net labels removed: VREG
- wire segments 53 -> 69
Other:
- moved on the sheet: JP2

Commit message: WIP of Rev 0.2
Parts:
- removed P1: CONN_01X09, Pin_Headers:Pin_Header_Straight_1x09, symbol CONN_01X09
- added Dflybk, Dvin: D_Schottky_Small, symbol D_Schottky_Small
- added L1: INDUCTOR_SMALL, symbol INDUCTOR_SMALL
- added Pbat: JST PH, w_conn_jst-ph:b2b-ph-kl, symbol CONN_01X02
- added Rsense: R_Small, symbol R_Small
- added Wgnd, Wvfb: TEST_1P, pcb_test_points:KEYSTONE_5016_PCB_Test_Point, symbol TEST_1P
- gave numbers to parts that had none: 2
- renumbered W2 to Wshdn, W1 to Wvreg
Connections:
- net GND: now also JP2.1, Dflybk.2 (A), Pbat.2 (P2), Wgnd.1
- net VIN: now also Dvin.1 (K); no longer CON1.1
- net at U1.10 (SENSE): now also Rsense.2
- net at Cbs.2, U1.12 (SW): now also Dflybk.1 (K), L1.1
- net at RV?.2, U1.7 (VFB): now also Wvfb.1
- net at U1.8 (NTC): no longer RV?.3
- net at C3.1, Dbatbst.2 (A), U1.9 (BAT): now also RV?.3, Pbat.1 (P1)
- net TIMER: no longer names the net of JP2.2, U1.6 (TIMER)
- new net: CON1.1, Dvin.2 (A)
- new net: L1.2, Rsense.1
- no-connect marks 1 -> 2
Other:
- moved on the sheet: C3, C?, Cbs, JP2, RV?

Commit message: WIP on Rev 0.2
Parts:
- added Wbat, Wsw: TEST_1P, pcb_test_points:KEYSTONE_5016_PCB_Test_Point, symbol TEST_1P
- L1: value INDUCTOR_SMALL -> 10uH
- Rsense: value R_Small -> 250mO
Connections:
- net at Rsense.2, U1.10 (SENSE): now also C3.1, Dbatbst.2 (A), Pbat.1 (P1), RV?.3, U1.9 (BAT), Wbat.1
- net at L1.2, Rsense.1: now also Wsw.1
Changed lines of the file:
@@
 P 6450 2750
 F 0 "L1" H 6450 2850 50  0000 C CNN
-F 1 "INDUCTOR_SMALL" H 6450 2700 50  0000 C CNN
+F 1 "10uH" H 6450 2700 50  0000 C CNN
 F 2 "" H 6450 2750 50  0000 C CNN
 F 3 "" H 6450 2750 50  0000 C CNN
@@
 P 6775 2975
 F 0 "Rsense" H 6805 2995 50  0000 L CNN
-F 1 "R_Small" H 6805 2935 50  0000 L CNN
+F 1 "250mO" H 6805 2935 50  0000 L CNN
 F 2 "" H 6775 2975 50  0000 C CNN
 F 3 "" H 6775 2975 50  0000 C CNN
@@
 Connection ~ 6100 3550
 Wire Wire Line
-	5950 3350 6775 3350
+	5950 3350 6900 3350
 Wire Wire Line
 	6775 3350 6775 3075
@@
 Wire Wire Line
 	4925 2825 4925 3050
+Wire Wire Line
+	6900 3350 6900 3550
+Connection ~ 6900 3550
+Connection ~ 6775 3350
+$Comp
+L TEST_1P Wbat
+U 1 1 56CEBC53
+P 7150 3475
+F 0 "Wbat" H 7150 3745 50  0000 C CNN
+F 1 "TEST_1P" H 7150 3675 50  0000 C CNN
+F 2 "pcb_test_points:KEYSTONE_5016_PCB_Test_Point" H 7350 3475 50  0001 C CNN
+F 3 "" H 7350 3475 50  0000 C CNN
+	1    7150 3475
+	1    0    0    -1
+$EndComp
+Wire Wire Line
+	7150 3475 7150 3550
+Connection ~ 7150 3550
+$Comp
+L TEST_1P Wsw
+U 1 1 56CEC1FA
+P 7100 2800
+F 0 "Wsw" H 7100 3070 50  0000 C CNN
+F 1 "TEST_1P" H 7100 3000 50  0000 C CNN
+F 2 "pcb_test_points:KEYSTONE_5016_PCB_Test_Point" H 7300 2800 50  0001 C CNN
+F 3 "" H 7300 2800 50  0000 C CNN
+	1    7100 2800
+	0    1    1    0
+$EndComp
+Wire Wire Line
+	7100 2800 6775 2800
+Connection ~ 6775 2800
 $EndSCHEMATC

Commit message: WIP on Rev 0.2
Parts:
- removed RV?: POT, bourns_trim_pots:Bourns_3362P_Trimmer, symbol POT
- removed Rsense: 250mO, symbol R_Small
- removed Wvfb: TEST_1P, pcb_test_points:KEYSTONE_5016_PCB_Test_Point, symbol TEST_1P
- added C4: 20pF, symbol C_Small
- added Pled: CONN_01X03, symbol CONN_01X03
- added Pload1: JST PH, w_conn_jst-ph:b2b-ph-kl, symbol CONN_01X02
- added Rfb1: 90k, symbol R_Small
- added Rfb2: 330k, symbol R_Small
- added Rfb3: 179k, symbol R_Small
- added Rsense1: 250mO, symbol R_Small
- added SWchrg1, SWflt1: Switch_SPDT_x2, symbol Switch_SPDT_x2
- added Wvfb1: TEST_1P, symbol TEST_1P
- gave numbers to parts that had none: 1
- renumbered Cbs to Cbs1, Dbatbst to Dbatbst1, Dflybk to Dflybk1, Dvin to Dvin1, L1 to Lsw1, Pbat to Pbat1, Wbat to Wbat1, Wgnd to Wgnd1, Wshdn to Wshdn1, Wsw to Wsw1
Connections:
- net GND: now also D1.2 (A), D2.2 (A), Pled.1 (P1), Pload1.2 (P2), Rfb2.2
- net VIN: no longer R1.2, R2.2
- net at C3.1, Dbatbst1.2 (A), Pbat1.1 (P1)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: now also C4.1, Pload1.1 (P1), Rfb1.1, Rsense1.2; no longer U1.10 (SENSE)
- net at U1.4 (~CHRG): now also R1.1; no longer D1.1 (K)
- net at U1.5 (~FAULT): now also R2.1; no longer D2.1 (K)
- net at U1.7 (VFB): now also C4.2, Rfb3.2, Wvfb1.1
- net at Lsw1.2, Wsw1.1: now also U1.10 (SENSE), Rsense1.1
- new net: D1.1 (K), SWchrg1.1 (A)
- new net: D2.1 (K), SWflt1.1 (A)
- new net: R1.2, SWchrg1.2 (B)
- new net: R2.2, SWflt1.2 (B)
- new net: Rfb1.2, Rfb2.1, Rfb3.1
- new net: Pled.2 (P2), SWflt1.3 (C)
- new net: Pled.3 (P3), SWchrg1.3 (C)
Other:
- note added: "4.2V FLT"
- note added: "400mA"
- moved on the sheet: D1, D2, Dbatbst1, R1, R2, Wbat1, Wshdn1, Wsw1

Commit message: WIP on Rev 0.2
Parts:
- removed C1: CTRIM, symbol CTRIM
- removed Dflybk1, Dvin1: D_Schottky_Small, symbol D_Schottky_Small
- removed SWchrg1, SWflt1: Switch_SPDT_x2, symbol Switch_SPDT_x2
- added C1: C_Small, Capacitors_SMD:C_0603_HandSoldering, symbol C_Small
- added Cbat1: 100uF, Capacitors_ThroughHole:C_Radial_D5_L6_P2.5, symbol CP1_Small
- added Dflybk1: ZLLS500, diodes:DIODES_INC_ZLLS500, symbol D_Schottky_Small_ZLLS500
- added Dvin1: D_Schottky_Small_ZLLS500, diodes:DIODES_INC_ZLLS500, symbol D_Schottky_Small_ZLLS500
- added JP2, JP3: JUMPER3, Pin_Headers:Pin_Header_Straight_1x03, symbol JUMPER3
- added Pload2: USB_A, connectors:WURTH_ELEKTRONIK_629104151021, symbol USB_A
- Cvfbat1: renamed from C4; footprint (none) -> Capacitors_SMD:C_0603_HandSoldering
- Dbatbst1: footprint (none) -> Diodes_ThroughHole:Diode_DO-35_SOD27_Horizontal_RM10
- Lsw1: footprint (none) -> inductors:PANASONIC_ELC09D100F
- Pled1: renamed from Pled; footprint (none) -> Pin_Headers:Pin_Header_Straight_1x03
- Rfb1, Rfb2, Rfb3, Rsense1: footprint (none) -> Resistors_SMD:R_0603_HandSoldering
- Wbat1, Wgnd1, Wshdn1, Wsw1: footprint pcb_test_points:KEYSTONE_5016_PCB_Test_Point -> pcb_test_points:HARWIN_S1751-46
- Wvfb1: footprint (none) -> pcb_test_points:HARWIN_S1751-46
- Wvreg1: renamed from Wvreg; footprint pcb_test_points:KEYSTONE_5016_PCB_Test_Point -> pcb_test_points:HARWIN_S1751-46
- renumbered C2 to Cvin2, JP2 to JP1
Connections:
- net GND: now also C1.2, Cbat1.2, Dflybk1.3 (A), Pload2.4 (GND)
- net VIN: now also Dvin1.1 (K); no longer RV1.1, RV2.1
- net SENSE: now reaches Lsw1.2, Rsense1.1, U1.10 (SENSE), Wsw1.1
- net BOOST: now reaches Cbs1.1, Dbatbst1.1 (K), U1.11 (BOOST)
- net SW: now reaches Cbs1.2, Lsw1.1, U1.12 (SW)
- net SW: now also Dflybk1.1 (K)
- net VFB: now reaches Cvfbat1.2, Rfb3.2, U1.7 (VFB), Wvfb1.1
- net BAT: now reaches C3.1, Cvfbat1.1, Dbatbst1.2 (A), Pbat1.1 (P1), Pload1.1 (P1), Rfb1.1, Rsense1.2, U1.9 (BAT), Wbat1.1
- net BAT: now also Cbat1.1, Pload2.1 (VCC)
- net at D1.1 (K): now also JP3.1
- net at D2.1 (K): now also JP2.1
- net at R1.2: now also JP3.2
- net at R2.2: now also JP2.2
- net at JP1.3: now also C1.1
- net at CON1.1: now also RV1.1, RV2.1, Dvin1.3 (A)
- net at Pled1.2 (P2): now also JP2.3
- net at Pled1.3 (P3): now also JP3.3
- no-connect marks 2 -> 5
