File: lt3652_breakout/lt3652_breakout.sch (KiCad schematic (older format))
At the start: 37 parts, among them U1 LT3652

Commit message: Upload of Rev 0.3
Parts:
- added Pslr2: JST PH, w_conn_jst-ph:b2b-ph-kl, symbol CONN_01X02
- added Rshdn1, Rvrg1: 10K, Resistors_SMD:R_0603_HandSoldering, symbol R_Small
- Dbatbst1: footprint Diodes_ThroughHole:Diode_DO-41_SOD81_Vertical_AnodeUp -> Diodes_ThroughHole:Diode_DO-35_SOD27_Horizontal_RM10
- R1, R2: value 220 -> 10K
- U1: footprint lt3652:LT3652MSE -> lt3652:LT3652MSE_HandSoldering
Connections:
- net BAT: now also Pbat1.1 (P1)
- net GND: now also Pslr2.2 (P2), Rshdn1.2, Rvrg1.2; no longer D1.2 (A), D2.2 (A), Pled1.1 (P1), RV1.3, RV2.3
- net VIN: now also D1.2 (A), D2.2 (A), Pled1.1 (P1)
- net at Dvin1.3 (A), Pslr1.1 (P1), RV1.1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: now also Pslr2.1 (P1)
- net at Cbat1.1, JPload1.2, Pload1.1 (P1)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: no longer Pbat1.1 (P1)
- new net: RV1.3, Rvrg1.1
- new net: RV2.3, Rshdn1.1
Other:
- moved on the sheet: Pbat1
Changed lines of the file:
@@
 F 0 "U1" H 5500 4100 60  0000 C CNN
 F 1 "LT3652" H 5500 4000 60  0000 C CNN
-F 2 "lt3652:LT3652MSE" H 5500 3450 60  0001 C CNN
+F 2 "lt3652:LT3652MSE_HandSoldering" H 5500 3450 60  0001 C CNN
 F 3 "" H 5500 3450 60  0000 C CNN
 	1    5500 3450
@@
 P 4900 3550
 F 0 "R1" H 4775 3500 50  0000 L CNN
-F 1 "220" V 4900 3500 39  0000 L CNN
+F 1 "10K" V 4900 3500 39  0000 L CNN
 F 2 "Resistors_SMD:R_0603_HandSoldering" H 4900 3550 50  0001 C CNN
 F 3 "" H 4900 3550 50  0000 C CNN
@@
 P 4900 3700
 F 0 "R2" H 4950 3650 50  0000 L CNN
-F 1 "220" V 4900 3650 39  0000 L CNN
+F 1 "10K" V 4900 3650 39  0000 L CNN
 F 2 "Resistors_SMD:R_0603_HandSoldering" H 4900 3700 50  0001 C CNN
 F 3 "" H 4900 3700 50  0000 C CNN
@@
 Connection ~ 4925 3050
 Wire Wire Line
-	5050 2375 4925 2375
+	4925 2375 5050 2375
 Connection ~ 4925 2375
 Wire Wire Line
@@
 L GND #PWR07
 U 1 1 56C6475C
-P 3750 3525
-F 0 "#PWR07" H 3750 3275 50  0001 C CNN
-F 1 "GND" H 3750 3375 50  0000 C CNN
-F 2 "" H 3750 3525 50  0000 C CNN
-F 3 "" H 3750 3525 50  0000 C CNN
-	1    3750 3525
-	1    0    0    -1
-$EndComp
-Wire Wire Line
-	3625 3450 3750 3525
+P 3625 3880
+F 0 "#PWR07" H 3625 3630 50  0001 C CNN
+F 1 "GND" H 3625 3730 50  0000 C CNN
+F 2 "" H 3625 3880 50  0000 C CNN
+F 3 "" H 3625 3880 50  0000 C CNN
+	1    3625 3880
+	1    0    0    -1
+$EndComp
+Wire Wire Line
+	3625 3450 3625 3520
 $Comp
 L POT RV2
@@
 	3950 3250 3950 2950
 Connection ~ 3950 2950
-$Comp
-L GND #PWR08
-U 1 1 56C65476
-P 3950 3800
-F 0 "#PWR08" H 3950 3550 50  0001 C CNN
-F 1 "GND" H 3950 3650 50  0000 C CNN
-F 2 "" H 3950 3800 50  0000 C CNN
-F 3 "" H 3950 3800 50  0000 C CNN
-	1    3950 3800
-	1    0    0    -1
-$EndComp
-Wire Wire Line
-	3950 3750 3950 3800
 Wire Wire Line
 	3625 2950 4100 2950
@@
 SHDN
 $Comp
-L GND #PWR09
+L GND #PWR08
 U 1 1 56C670F4
-P 8055 3700
-F 0 "#PWR09" H 8055 3450 50  0001 C CNN
-F 1 "GND" H 8055 3550 50  0000 C CNN
-F 2 "" H 8055 3700 50  0000 C CNN
-F 3 "" H 8055 3700 50  0000 C CNN
-	1    8055 3700
+P 7630 4110
+F 0 "#PWR08" H 7630 3860 50  0001 C CNN
+F 1 "GND" H 7630 3960 50  0000 C CNN
+F 2 "" H 7630 4110 50  0000 C CNN
+F 3 "" H 7630 4110 50  0000 C CNN
+	1    7630 4110
 	1    0    0    -1
 $EndComp
@@
 F 0 "Dbatbst1" H 6200 3280 50  0000 L CNN
 F 1 "D_Small" H 6100 3120 50  0000 L CNN
-F 2 "Diodes_ThroughHole:Diode_DO-41_SOD81_Vertical_AnodeUp" V 6250 3200 50  0001 C CNN
+F 2 "Diodes_ThroughHole:Diode_DO-35_SOD27_Horizontal_RM10" V 6250 3200 50  0001 C CNN
 F 3 "" V 6250 3200 50  0000 C CNN
 	1    6250 3200
@@
 L CONN_01X02 Pbat1
 U 1 1 56CB9AD3
-P 8330 3600
-F 0 "Pbat1" H 8330 3750 50  0000 C CNN
-F 1 "JST PH" V 8430 3600 50  0000 C CNN
-F 2 "w_conn_jst-ph:b2b-ph-kl" H 8330 3600 50  0001 C CNN
-F 3 "" H 8330 3600 50  0000 C CNN
-	1    8330 3600
-	1    0    0    -1
-$EndComp
-Wire Wire Line
-	8055 3700 8055 3650
-Wire Wire Line
-	8055 3650 8130 3650
+P 7905 4010
+F 0 "Pbat1" H 7905 4160 50  0000 C CNN
+F 1 "JST PH" V 8005 4010 50  0000 C CNN
+F 2 "w_conn_jst-ph:b2b-ph-kl" H 7905 4010 50  0001 C CNN
+F 3 "" H 7905 4010 50  0000 C CNN
+	1    7905 4010
+	1    0    0    -1
+$EndComp
+Wire Wire Line
+	7630 4110 7630 4060
+Wire Wire Line
+	7630 4060 7705 4060
 Wire Wire Line
 	5950 3050 5950 2750
@@
 	6275 2400 6100 2400
 $Comp
-L GND #PWR010
+L GND #PWR09
 U 1 1 56CBB710
 P 6775 2475
-F 0 "#PWR010" H 6775 2225 50  0001 C CNN
+F 0 "#PWR09" H 6775 2225 50  0001 C CNN
 F 1 "GND" H 6775 2325 50  0000 C CNN
 F 2 "" H 6775 2475 50  0000 C CNN
@@
 Connection ~ 6750 3850
 $Comp
-L GND #PWR011
+L GND #PWR010
 U 1 1 56CF50A1
 P 6750 4200
-F 0 "#PWR011" H 6750 3950 50  0001 C CNN
+F 0 "#PWR010" H 6750 3950 50  0001 C CNN
 F 1 "GND" H 6750 4050 50  0000 C CNN
 F 2 "" H 6750 4200 50  0000 C CNN
@@
 	8080 3150 8680 3150
 $Comp
-L GND #PWR012
+L GND #PWR011
 U 1 1 56CF694F
 P 8630 3400
-F 0 "#PWR012" H 8630 3150 50  0001 C CNN
+F 0 "#PWR011" H 8630 3150 50  0001 C CNN
 F 1 "GND" H 8630 3250 50  0000 C CNN
 F 2 "" H 8630 3400 50  0000 C CNN
@@
 Wire Wire Line
 	3365 4085 4565 4085
-$Comp
-L GND #PWR013
-U 1 1 56D0CA13
-P 2515 4770
-F 0 "#PWR013" H 2515 4520 50  0001 C CNN
-F 1 "GND" H 2515 4620 50  0000 C CNN
-F 2 "" H 2515 4770 50  0000 C CNN
-F 3 "" H 2515 4770 50  0000 C CNN
-	1    2515 4770
-	1    0    0    -1
-$EndComp
 Wire Wire Line
 	2855 4185 3070 4185
@@
 $EndComp
 $Comp
-L GND #PWR014
+L GND #PWR012
 U 1 1 56D16B0E
 P 8555 2865
-F 0 "#PWR014" H 8555 2615 50  0001 C CNN
+F 0 "#PWR012" H 8555 2615 50  0001 C CNN
 F 1 "GND" H 8555 2715 50  0000 C CNN
 F 2 "" H 8555 2865 50  0000 C CNN
@@
 NoConn ~ 8615 2640
 NoConn ~ 9015 2940
-Connection ~ 8080 3150
 Wire Wire Line
 	8370 3170 8370 3150
@@
 $EndComp
 Wire Wire Line
-	7425 3550 5950 3550
+	5950 3550 7425 3550
 Wire Wire Line
 	6100 3925 6100 3550
@@
 Connection ~ 8080 2925
 Wire Wire Line
-	8080 3550 8130 3550
-Wire Wire Line
-	7360 3550 7360 3175
+	7360 3175 7360 3960
 Wire Wire Line
 	7360 3175 7880 3175
 Connection ~ 7360 3550
 Wire Wire Line
-	7625 3550 7625 2140
-Wire Wire Line
-	7625 2140 5385 2140
+	7625 2140 7625 3550
+Wire Wire Line
+	5385 2140 7625 2140
 Wire Wire Line
 	7880 2675 7625 2675
 Connection ~ 7625 2675
-Wire Wire Line
-	8080 2440 8080 3550
-$Comp
-L PWR_FLAG #FLG015
+$Comp
+L PWR_FLAG #FLG013
 U 1 1 56D7B958
 P 8315 2400
-F 0 "#FLG015" H 8315 2495 50  0001 C CNN
+F 0 "#FLG013" H 8315 2495 50  0001 C CNN
 F 1 "PWR_FLAG" H 8315 2580 50  0000 C CNN
 F 2 "" H 8315 2400 50  0000 C CNN
@@
 	8315 2400 8315 2440
 Connection ~ 8315 2440
+$Comp
+L CONN_01X02 Pslr2
+U 1 1 56D8B1A1
+P 4430 1940
+F 0 "Pslr2" H 4430 2090 50  0000 C CNN
+F 1 "JST PH" V 4530 1940 50  0000 C CNN
+F 2 "w_conn_jst-ph:b2b-ph-kl" H 4430 1940 50  0001 C CNN
+F 3 "" H 4430 1940 50  0000 C CNN
+	1    4430 1940
+	0    1    -1   0
+$EndComp
+Wire Wire Line
+	4480 2140 4480 2190
+Wire Wire Line
+	4480 2190 4925 2190
+Connection ~ 4925 2190
+Wire Wire Line
+	4380 2140 4380 2375
+Connection ~ 4380 2375
+Text Label 2515 4740 3    60   ~ 0
+VIN
+$Comp
+L R_Small Rvrg1
+U 1 1 56D9C63D
+P 3625 3620
+F 0 "Rvrg1" H 3655 3640 50  0000 L CNN
+F 1 "10K" H 3655 3580 50  0000 L CNN
+F 2 "Resistors_SMD:R_0603_HandSoldering" H 3625 3620 50  0001 C CNN
+F 3 "" H 3625 3620 50  0000 C CNN
+	1    3625 3620
+	1    0    0    -1
+$EndComp
+$Comp
+L R_Small Rshdn1
+U 1 1 56D9CD10
+P 3815 3805
+F 0 "Rshdn1" H 3845 3825 50  0000 L CNN
+F 1 "10K" H 3845 3765 50  0000 L CNN
+F 2 "Resistors_SMD:R_0603_HandSoldering" H 3815 3805 50  0001 C CNN
+F 3 "" H 3815 3805 50  0000 C CNN
+	1    3815 3805
+	0    1    1    0
+$EndComp
+Wire Wire Line
+	3625 3720 3625 3880
+Wire Wire Line
+	3715 3805 3625 3805
+Connection ~ 3625 3805
+Wire Wire Line
+	3950 3750 3950 3805
+Wire Wire Line
+	3950 3805 3915 3805
+Wire Wire Line
+	8080 2440 8080 3150
+Wire Wire Line
+	7360 3960 7705 3960
 $EndSCHEMATC
